File: eagle/projects/ch340_usb_3/ch340_usb.brd (EAGLE design)
At the start: 40.6 x 54.4 mm, 27 parts, among them J1 1734035-4, U1 HX711, U2 LM393, U3 AMS1117, X1 CSM-7X-DU

Commit message: 150324
Routing:
- net 3V3: track 163.4 -> 160.2 mm
- net GND: track 21.8 -> 19.8 mm
- net N$9: track 0.00 -> 2.00 mm
- net N$8: track 0.00 -> 2.00 mm
- net N$7: track 0.00 -> 2.00 mm
- net N$6: track 0.00 -> 2.00 mm
- net N$5: track 0.00 -> 2.00 mm
- net N$12: track 0.00 -> 2.00 mm
- net N$11: track 0.00 -> 2.00 mm
- net N$10: track 0.00 -> 2.00 mm
Changed lines of the file:
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@@
 <setting verticaltext="up"/>
 </settings>
-<grid distance="25" unitdist="mil" unit="mil" style="lines" multiple="1" display="yes" altdistance="1" altunitdist="mil" altunit="mil"/>
+<grid distance="9.84251969" unitdist="mil" unit="mil" style="lines" multiple="1" display="yes" altdistance="1" altunitdist="mil" altunit="mil"/>
 <layers>
 <layer number="1" name="Top" color="4" fill="1" visible="yes" active="yes"/>
@@
 <layer number="43" name="vRestrict" color="2" fill="10" visible="no" active="yes"/>
 <layer number="44" name="Drills" color="7" fill="1" visible="no" active="yes"/>
-<layer number="45" name="Holes" color="7" fill="1" visible="yes" active="yes"/>
+<layer number="45" name="Holes" color="7" fill="1" visible="no" active="yes"/>
 <layer number="46" name="Milling" color="3" fill="1" visible="no" active="yes"/>
 <layer number="47" name="Measures" color="7" fill="1" visible="no" active="yes"/>
@@
 </layers>
 <board>
-<fusionsync huburn="a.YnVzaW5lc3M6bXlvZ3I0NDE" projecturn="a.YnVzaW5lc3M6bXlvZ3I0NDEjRDIwMjAxMDA0MzM5Mzc1ODc2" f3durn="urn:adsk.wipprod:dm.lineage:P4YMTViJTeS0FxHuX-nNnA" pcbguid="d9dcfa45-c09e-4eee-8e59-c28738228a45" lastpulledtime="" lastsyncedchangeguid="" latestrevisionid="38992e13-cc54-4ef7-9ff4-9eadfa1cea1e" lastsyncedrevisionid="38992e13-cc54-4ef7-9ff4-9eadfa1cea1e" lastboardhashguid="e37499c2-fadb-361a-f74a-95f53673bdbc" lastpushedtime="2023-03-27T17:05:00Z" linktopcb3d="true"/>
+<fusionsync huburn="a.YnVzaW5lc3M6bXlvZ3I0NDE" projecturn="a.YnVzaW5lc3M6bXlvZ3I0NDEjRDIwMjAxMDA0MzM5Mzc1ODc2" f3durn="urn:adsk.wipprod:dm.lineage:P4YMTViJTeS0FxHuX-nNnA" pcbguid="" lastpulledtime="" lastsyncedchangeguid="" latestrevisionid="38992e13-cc54-4ef7-9ff4-9eadfa1cea1e" lastsyncedrevisionid="38992e13-cc54-4ef7-9ff4-9eadfa1cea1e" lastboardhashguid="e37499c2-fadb-361a-f74a-95f53673bdbc" lastpushedtime="2023-03-27T17:05:00Z" linktopcb3d="true"/>
 <plain>
-<wire x1="0" y1="0" x2="40.64" y2="0" width="0" layer="20"/>
-<wire x1="40.64" y1="0" x2="40.64" y2="54.407" width="0" layer="20"/>
-<wire x1="40.64" y1="54.407" x2="0" y2="54.407" width="0" layer="20"/>
-<wire x1="0" y1="54.407" x2="0" y2="0" width="0" layer="20"/>
+<wire x1="0" y1="0" x2="40.64" y2="0" width="0.254" layer="20"/>
+<wire x1="40.64" y1="0" x2="40.64" y2="54.407" width="0.254" layer="20"/>
+<wire x1="40.64" y1="54.407" x2="0" y2="54.407" width="0.254" layer="20"/>
+<wire x1="0" y1="54.407" x2="0" y2="0" width="0.254" layer="20"/>
 <text x="3.175" y="27.94" size="1.27" layer="25">JP1</text>
 <text x="3.175" y="18.415" size="1.27" layer="25">JP2</text>
@@
 <circle x="18.1102" y="49.149" radius="0.5588" width="0.254" layer="25"/>
 <circle x="22.5298" y="49.149" radius="0.5588" width="0.254" layer="25"/>
+<wire x1="0.25" y1="51" x2="3.25" y2="54" width="0.0254" layer="41"/>
+<wire x1="3.5" y1="0.25" x2="0.25" y2="3.5" width="0.0254" layer="41"/>
+<wire x1="40.75" y1="50.5" x2="37" y2="54.25" width="0.0254" layer="41"/>
 </plain>
 <attributes>
@@
 <param name="mdViaViaSameLayer" value="6mil"/>
 <param name="mnLayersViaInSmd" value="2"/>
-<param name="mdCopperDimension" value="0mil"/>
+<param name="mdCopperDimension" value="1mm"/>
 <param name="mdDrill" value="6mil"/>
 <param name="mdSmdStop" value="0mil"/>
@@
 <param name="srMaxRoundness" value="0mil"/>
 <param name="slThermalIsolate" value="10mil"/>
-<param name="slThermalsForVias" value="0"/>
+<param name="slThermalsForVias" value="1"/>
 <param name="dpMaxLengthDifference" value="10mm"/>
 <param name="dpGapFactor" value="2.5"/>
@@
 <wire x1="18.72" y1="44.755" x2="18.415" y2="44.45" width="0.254" layer="1"/>
 <contactref element="C7" pad="2"/>
-<wire x1="26.4" y1="41.91" x2="27.559" y2="41.91" width="0.254" layer="1"/>
-<wire x1="27.559" y1="41.91" x2="28.194" y2="42.545" width="0.254" layer="1"/>
 <via x="28.194" y="42.545" extent="1-16" drill="0.6" diameter="1.2"/>
 <wire x1="28.194" y1="42.545" x2="28.194" y2="46.99" width="0.254" layer="16"/>
@@
 <wire x1="10.795" y1="36.195" x2="8.89" y2="34.29" width="0.254" layer="1"/>
 <wire x1="8.89" y1="34.29" x2="8.89" y2="23.495" width="0.254" layer="1"/>
-<wire x1="39.37" y1="14.605" x2="39.37" y2="13.97" width="0.6096" layer="1"/>
-<wire x1="39.37" y1="13.97" x2="39.37" y2="8.89" width="0.6096" layer="1"/>
-<wire x1="39.37" y1="8.89" x2="39.37" y2="3.175" width="0.6096" layer="1"/>
-<wire x1="39.37" y1="3.175" x2="38.1" y2="1.905" width="0.6096" layer="1"/>
+<wire x1="39.12" y1="3.425" x2="37.6" y2="1.905" width="0.6096" layer="1"/>
 <wire x1="24.765" y1="9.525" x2="24.765" y2="13.97" width="0.6096" layer="1"/>
 <wire x1="24.765" y1="13.97" x2="23.495" y2="15.24" width="0.6096" layer="1"/>
-<wire x1="38.1" y1="1.905" x2="32.385" y2="1.905" width="0.6096" layer="1"/>
+<wire x1="37.6" y1="1.905" x2="32.385" y2="1.905" width="0.6096" layer="1"/>
 <wire x1="32.385" y1="1.905" x2="24.765" y2="9.525" width="0.6096" layer="1"/>
 <wire x1="23.495" y1="15.24" x2="22.479" y2="15.24" width="0.6096" layer="1"/>
@@
 <wire x1="12.7" y1="15.655" x2="16.51" y2="15.655" width="0.4064" layer="1"/>
 <wire x1="18.415" y1="14.09189375" x2="19.56310625" y2="15.24" width="0.6096" layer="1"/>
-<wire x1="37.465" y1="14.285" x2="39.05" y2="14.285" width="0.254" layer="1"/>
-<wire x1="39.05" y1="14.285" x2="39.37" y2="14.605" width="0.254" layer="1"/>
-<wire x1="37.465" y1="14.285" x2="39.055" y2="14.285" width="0.254" layer="1"/>
-<wire x1="39.055" y1="14.285" x2="39.37" y2="13.97" width="0.254" layer="1"/>
-<wire x1="37.465" y1="9.078" x2="39.182" y2="9.078" width="0.254" layer="1"/>
-<wire x1="39.182" y1="9.078" x2="39.37" y2="8.89" width="0.254" layer="1"/>
 <wire x1="23.92" y1="40.005" x2="29.845" y2="40.005" width="0.4064" layer="1"/>
 <wire x1="12.7" y1="34.02" x2="12.7" y2="36.195" width="0.254" layer="1"/>
 <wire x1="32.385" y1="38.176" x2="31.191" y2="39.37" width="0.6096" layer="1"/>
 <wire x1="29.921" y1="39.37" x2="31.191" y2="39.37" width="0.6096" layer="1"/>
-<wire x1="32.385" y1="26.67" x2="39.37" y2="19.685" width="0.6096" layer="1"/>
-<wire x1="39.37" y1="19.685" x2="39.37" y2="14.605" width="0.6096" layer="1"/>
+<wire x1="32.385" y1="26.67" x2="39.12" y2="19.935" width="0.6096" layer="1"/>
 <wire x1="32.385" y1="38.176" x2="32.385" y2="34.29" width="0.6096" layer="1"/>
 <wire x1="32.385" y1="34.29" x2="32.385" y2="31.75" width="0.6096" layer="1"/>
@@
 <wire x1="24.4" y1="40.783" x2="24.4" y2="41.91" width="0.254" layer="1"/>
 <wire x1="24.13" y1="40.513" x2="24.4" y2="40.783" width="0.254" layer="1"/>
+<wire x1="39.12" y1="19.935" x2="39.12" y2="14.25" width="0.6096" layer="1"/>
+<wire x1="39.12" y1="14.25" x2="39.12" y2="9" width="0.6096" layer="1"/>
+<wire x1="39.12" y1="9" x2="39.12" y2="3.425" width="0.6096" layer="1"/>
+<wire x1="37.465" y1="14.285" x2="39.085" y2="14.285" width="0.254" layer="1"/>
+<wire x1="39.085" y1="14.285" x2="39.12" y2="14.25" width="0.254" layer="1"/>
+<wire x1="37.465" y1="9.078" x2="39.042" y2="9.078" width="0.254" layer="1"/>
+<wire x1="39.042" y1="9.078" x2="39.12" y2="9" width="0.254" layer="1"/>
 <wire x1="34.56" y1="34.29" x2="36.1188" y2="39.37" width="0" layer="19" extent="1-1"/>
 <wire x1="29.845" y1="40.005" x2="29.921" y2="39.37" width="0" layer="19" extent="1-1"/>
@@
 <contactref element="D1" pad="A"/>
 <wire x1="21.92" y1="46.549" x2="21.92" y2="44.755" width="0.4064" layer="1"/>
-<wire x1="21.92" y1="44.755" x2="21.971" y2="44.704" width="0.4064" layer="1"/>
 <wire x1="21.971" y1="44.704" x2="22.225" y2="44.45" width="0.6096" layer="1"/>
 <wire x1="27.305" y1="44.45" x2="27.94" y2="45.085" width="0.6096" layer="1"/>
 <wire x1="27.94" y1="45.085" x2="29.85" y2="45.085" width="0.6096" layer="1"/>
 <wire x1="22.225" y1="44.45" x2="27.305" y2="44.45" width="0.6096" layer="1"/>
+<wire x1="21.971" y1="44.704" x2="21.92" y2="44.755" width="0" layer="19" extent="1-1"/>
 </signal>
 <signal name="N$1">
@@
 <wire x1="19.05" y1="2.159" x2="14.351" y2="2.159" width="0.254" layer="1"/>
 </signal>
+<signal name="N$5">
+<wire x1="1.2446" y1="54.094" x2="1.2446" y2="52.094" width="0.2" layer="1"/>
+</signal>
+<signal name="N$6">
+<wire x1="0.2446" y1="53.094" x2="2.2446" y2="53.094" width="0.2" layer="1"/>
+</signal>
+<signal name="N$7">
+<wire x1="39.4034" y1="54.1114" x2="39.4034" y2="52.1114" width="0.2" layer="1"/>
+</signal>
+<signal name="N$8">
+<wire x1="38.4034" y1="53.1114" x2="40.4034" y2="53.1114" width="0.2" layer="1"/>
+</signal>
+<signal name="N$9">
+<wire x1="1.2526" y1="2.2446" x2="1.2526" y2="0.2446" width="0.2" layer="1"/>
+</signal>
+<signal name="N$10">
+<wire x1="0.2526" y1="1.2446" x2="2.2526" y2="1.2446" width="0.2" layer="1"/>
+</signal>
+<signal name="N$11">
+<wire x1="39.4234" y1="2.2218" x2="39.4234" y2="0.2218" width="0.2" layer="1"/>
+</signal>
+<signal name="N$12">
+<wire x1="38.4234" y1="1.2218" x2="40.4234" y2="1.2218" width="0.2" layer="1"/>
+</signal>
 </signals>
