File: eagle/projects/cypd3177/StaticPlatformMain_v1.sch (EAGLE design)
At the start: 27 parts, among them J1 1734035-4, U1 HX711, U2 LM393, U3 AMS1117, X1 CSM-7X-DU

Commit message: 150324
Parts:
- removed C7: 100n, rcl:C-EUC0805K
- removed D1: BAT60B, diode:MBR0520LT
- removed DTR, RTS, RX, TX: PWR, led:LEDCHIPLED_0805
- removed J1: 1734035-4, USB connector:1734035-4
- removed J2: (no value), con-lstb_round_pads:MA06-1
- removed U$1: DIPSW4, dipsw:DIPSW4
- removed X1: CSM-7X-DU, crystal:CSM-7X-DU
- added C10: 10u, rcl:C-EUC0805
- added C301, C304, C310, C311: 1u, rcl:C-EUC0805K
- added C302, C303: 100n, rcl:C-EUC0805K
- added D2: 9V, BZV55C12_L0G:BZV55C12_L0G
- added FAULT, PWR: GREEN, adafruit:LEDCHIPLED_0805
- added J5: USB4105-GF-A, USB4105-GF-A:USB4105-GF-A
- added JTAG: CORTEX_DEBUG_SMD, SparkFun-Connectors:CORTEX_DEBUG_SMD
- added LED: RED, adafruit:LEDCHIPLED_0805
- added Q1, Q2: DMP3098LSD-13, DMP3098LSD-13:DMP3098LSD-13
- added Q3: 2N7002, 2N7002:2N7002
- added R1, R11: 3k3, rcl:R-EU_R0805
- added R10, R12, R13, R14, R15, R16, R308: 0, rcl:R-EU_R0805
- added R17, R312: 10k, rcl:R-EU_R0805
- added R301, R303, R305: 5k1, rcl:R-EU_R0805
- added R302, R304, R306, R311, R320: 1k, rcl:R-EU_R0805
- added R307: 10M, rcl:R-EU_R0805
- added R310, R321: 50k, rcl:R-EU_R0805
- added RESET: MOMENTARY-SWITCH-SPST-SMD-6.0X3.5MM, SparkFun-Switches:MOMENTARY-SWITCH-SPST-SMD-6.0X3.5MM
- added SV1: (no value), con-lstb_round_pads:MA04-1
- added SV2: (no value), con-lstb_round_pads:MA05-2
- added TP1, TP2, TP3, TP4, TP5, TP6, TP7, TP8: TPTP18R, testpad:TPTP18R
- C1: value 10u -> 3u3
- C2: value 5u6 -> 10u, 6.3V
- C3: value 100n -> 4.7u, 6.3V
- C4: value 10n -> 1u, 6.3V
- C5: value 22p -> 100n, 6.3V
- C6: value 22p -> 1u, 6.3V; device rcl:C-EUC0805K -> rcl:C-EUC0805
- R3, R4, R5, R7: value 1k -> 2k2
- R6: value 1k -> 22k
- R8: value 1k -> 10k
- R9: value 1k -> 0
- U1: value HX711 -> ATSAMD21E18A; device ch340:CH340G -> SAMD21E18:ATSAMD21E18A-AUTQFP32_MC_MCH-M
- U2: value LM393 -> AMS1117; device lm393:LM393 -> SparkFun-IC-Power:V_REG_LM1117SOT223
- U3: value AMS1117 -> CYPD3177-24LQXQT; device SparkFun-IC-Power:V_REG_LM1117SOT223 -> CYPD3177-24LQXQT:CYPD3177-24LQXQT
Connections:
- removed net /DTR: R6.2, U$1.2A, U2.OUTA
- removed net /RTS: R7.2, U$1.4A, U2.OUTB
- removed net CTS: U1.CTS
- removed net DCD: U1.DCD
- removed net DSR: U1.DSR
- removed net DTR: U$1.1A, U1.DTR, U2.INNA
- removed net DTR_O: J2.5, R3.2, U$1.1B, U$1.2B
- removed net D_N: J1.D-, U1.UDN
- removed net D_P: J1.D+, U1.UDP
- removed net RI: U1.RI
- removed net RS232: U1.R232
- removed net RTS: U$1.3A, U1.RTS, U2.INNB
- removed net RTS_O: J2.4, R2.2, U$1.3B, U$1.4B
- removed net RX: J2.3, R4.2, U1.RXD
- removed net TX: J2.2, R5.2, U1.TXD
- removed net USB_5V: C1.1, D1.C, U3.IN
- removed net VCC/2: R8.1, R9.2, U2.INPA, U2.INPB
- removed net XI: C5.1, U1.XI, X1.2
- removed net XO: C6.1, U1.XO, X1.1
- new net CC1: J5.CC1, TP7.TP, U3.CC1
- new net CC2: J5.CC2, TP8.TP, U3.CC2
- new net DTCT: JTAG.GNDDTCT
- new net FAULT: Q3.G, R6.1, U3.FAULT
- new net FLIP: R3.2, U3.FLIP
- new net G1G2: C310.2, C311.2, D2.A, Q1.G1, Q1.G2, R310.2, R311.1, R312.2, TP3.TP
- new net G3G4: Q2.G1, Q2.G2, R320.1, R321.2, TP4.TP
- new net KEY: JTAG.KEY
- new net LED: R11.2, U1.PA07
- new net LED_GP: LED.A, R11.1
- new net LED_PWR: PWR.A, R2.1
- new net N$10: R307.1, R308.2, U3.ISNK_FINE
- new net N$19: J5.SBU2
- new net N$24: JTAG.NC/TDI
- new net N$28: U1.PA10
- new net N$5: R305.1, R306.2, U3.ISNK_COARSE
- new net N$7: Q3.D, R1.2
- new net N$9: J5.SBU1
- new net P14: SV2.10, U1.PA11
- new net P15: SV2.9, U1.PA14
- new net P16: SV2.8, U1.PA15
- new net P17: SV2.7, U1.PA16
- new net P18: SV2.6, U1.PA17
- new net P19: SV2.5, U1.PA18
- new net P20: SV2.4, U1.PA19
- new net P21: SV2.3, U1.PA22
- new net P22: SV2.2, U1.PA23
- new net RESET: JTAG.!RESET, R8.1, RESET.1, U1.!RESET
- new net S1S2: D2.K, Q1.S1, Q1.S2, R310.1
- new net S3S4: Q2.S1, Q2.S2
- new net SAFE_PWR_EN: R320.2, U3.SAFE_PWR_EN
- new net SCL: R12.2, R5.2, U3.HPI_SCL
- new net SDA: R13.2, R4.2, U3.HPI_SDA
- new net SWCLK: JTAG.SWDCLK/TCK, R17.1, U1.PA30
- new net SWDIO: JTAG.SWDIO/TMS, U1.PA31
- new net SWO: JTAG.SWO/TDO
- new net USB_D_N: J5.DN1, J5.DN2, R9.1
- new net USB_D_P: J5.DP1, J5.DP2, R10.1
- new net VBUS_FET_EN: R311.2, U3.VBUS_FET_EN
- new net VCCD: C304.1, TP6.TP, U3.VCCD
- new net VDDCORE: C6.1, U1.VDDCORE
- new net VDDD: C301.1, C302.1, C303.1, TP5.TP, U3.VDDD
- new net VDDOUT: C2.1, C311.1, Q1.D1_1, Q1.D1_2, Q2.D2_1, Q2.D2_2, SV1.3, TP2.TP, U2.IN, U3.VDC_OUT
- new net _3V3: C10.1, JTAG.VCC, R14.1, R17.2, R8.2, U1.VDDANA, U1.VDDIN
- new net _GND: C10.2, C6.2, JTAG.GND@3, JTAG.GND@5, LED.C, R15.1, R16.1, RESET.2, SV2.1, U1.GND, U1.GND_2
- new net _SCL: R12.1, U1.PA09
- new net _SDA: R13.1, U1.PA08
- new net _USB_D_N: R9.2, U1.PA24
- new net _USB_D_P: R10.2, U1.PA25
- net 3V3: now also C5.1, R14.2, R2.2, R3.1, R301.2, R303.2, R305.2, R307.2, R4.1, R5.1, R7.2, SV1.2, U2.OUT, U2.OUT@1; no longer C2.1, C7.1, DTR.C, J2.6, R6.1, R7.1, R9.1, RTS.C, RX.C, TX.C, U1.V3, U1.VCC, U2.VCC, U3.OUT, U3.OUT@1
- net GND: now also C301.2, C302.2, C303.2, C304.2, J5.GND, J5.SHELL_GND, PWR.C, Q3.S, R15.2, R16.2, R302.1, R304.1, R306.1, R308.1, R6.2, SV1.1, U2.ADJ, U3.EP, U3.GND_1, U3.GND_2; no longer C6.2, C7.2, J1.GND, J1.SHIELD, J2.1, R8.2, U1.GND, U2.GND, U3.ADJ
- net N$1: now also FAULT.C, R1.1; no longer DTR.A, R3.1
- net N$2: now also R7.1, U3.HPI_INT; no longer R2.1, RTS.A
- net N$3: now also R301.1, R302.2, U3.VBUS_MIN; no longer R4.1, RX.A
- net N$4: now also R303.1, R304.2, U3.VBUS_MAX; no longer R5.1, TX.A
- net VBUS: now also C1.1, C310.1, FAULT.A, J5.VBUS, Q1.D2_1, Q1.D2_2, Q2.D1_1, Q2.D1_2, R312.1, R321.1, SV1.4, TP1.TP, U3.VBUS_IN; no longer D1.A, J1.VBUS
Other:
- note added: "uCONTROLLER"
- moved on the sheet: C1, C2, C3, C4, C5, C6, R2, R3, R4, R5, R6, R7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
