File: eagle/projects/static_platform_v1.1/StaticPlatformADC_v1.sch (EAGLE design)
At the start: 27 parts, among them J1 1734035-4, U1 HX711, U2 LM393, U3 AMS1117, X1 CSM-7X-DU

Commit message: 150324
Parts:
- removed D1: BAT60B, diode:MBR0520LT
- removed DTR, RTS, RX, TX: PWR, led:LEDCHIPLED_0805
- removed J2: (no value), con-lstb_round_pads:MA06-1
- removed R7, R8, R9: 1k, rcl:R-EU_R0805
- removed U$1: DIPSW4, dipsw:DIPSW4
- removed U2: LM393, lm393:LM393
- removed U3: AMS1117, SparkFun-IC-Power:V_REG_LM1117SOT223
- removed X1: CSM-7X-DU, crystal:CSM-7X-DU
- added C8, C9: 1u, 6.3V, rcl:C-EUC0805
- added GPIO: (no value), SparkFun-Connectors:CONN_08NO_SILK_FEMALE_PTH
- added JMP: (no value), SparkFun-Connectors:CONN_021X02_NO_SILK
- added L1: 3.3u, rcl:L-USL3225P
- added LOAD_CELL: (no value), SparkFun-Connectors:CONN_05NO_SILK
- added Q1: MMBT4403LT1SMD, transistor-pnp:MMBT4403LT1SMD
- added R1: 10k, rcl:R-EU_R0805
- C1: value 10u -> 100n, 6.3V; device rcl:C-EUC0805K -> rcl:C-EUC0805
- C2: value 5u6 -> 10u, 6.3V; device rcl:C-EUC0805K -> rcl:C-EUC0805
- C3: value 100n -> 10u, 6.3V; device rcl:C-EUC0805K -> rcl:C-EUC0805
- C4: value 10n -> 100n, 6.3V; device rcl:C-EUC0805K -> rcl:C-EUC0805
- C5: value 22p -> 100n, 6.3V; device rcl:C-EUC0805K -> rcl:C-EUC0805
- C6: value 22p -> 1u, 6.3V; device rcl:C-EUC0805K -> rcl:C-EUC0805
- C7: value 100n -> 100n, 6.3V; device rcl:C-EUC0805K -> rcl:C-EUC0805
- J1: value 1734035-4 -> DS1013-10SSIB1; device USB connector:1734035-4 -> IDC_CON_DS1013-10SSIB1:DS1013-10SSIB1
- R2: value 1k -> 20k
- R3: value 1k -> 8.2k
- R4, R5: value 1k -> 100
- U1: device ch340:CH340G -> HX711:HX711
Connections:
- removed net /DTR: R6.2, U$1.2A, U2.OUTA
- removed net /RTS: R7.2, U$1.4A, U2.OUTB
- removed net CTS: U1.CTS
- removed net DCD: U1.DCD
- removed net DSR: U1.DSR
- removed net DTR: U$1.1A, U1.DTR, U2.INNA
- removed net DTR_O: J2.5, R3.2, U$1.1B, U$1.2B
- removed net D_N: J1.D-, U1.UDN
- removed net D_P: J1.D+, U1.UDP
- removed net N$1: DTR.A, R3.1
- removed net N$2: R2.1, RTS.A
- removed net RI: U1.RI
- removed net RS232: U1.R232
- removed net RTS: U$1.3A, U1.RTS, U2.INNB
- removed net RTS_O: J2.4, R2.2, U$1.3B, U$1.4B
- removed net RX: J2.3, R4.2, U1.RXD
- removed net TX: J2.2, R5.2, U1.TXD
- removed net USB_5V: C1.1, D1.C, U3.IN
- removed net VBUS: D1.A, J1.VBUS
- removed net VCC/2: R8.1, R9.2, U2.INPA, U2.INPB
- removed net XI: C5.1, U1.XI, X1.2
- removed net XO: C6.1, U1.XO, X1.1
- new net A+: LOAD_CELL.4, R5.1
- new net A-: LOAD_CELL.3, R4.1
- new net E+: C3.1, L1.2, Q1.C, R2.1, U1.AVDD
- new net LC_CON: J1.9, JMP.1, R1.2
- new net LC_DOUT: J1.5, U1.DOUT
- new net LC_SCK: J1.7, U1.PD_SCK
- new net N$10: GPIO.7, R6.2
- new net N$12: C4.1, R4.2, U1.INA-
- new net N$13: C4.2, R5.2, U1.INA+
- new net N$16: J1.6
- new net N$5: R2.2, R3.1, U1.VFB
- new net N$7: C1.2, U1.VBG
- new net N$8: J1.4
- new net SCL: GPIO.2, J1.10
- new net SDA: GPIO.1, J1.8
- new net TEMP: C7.1, J1.3, R6.1
- net 3V3: now also C8.1, C9.2, GPIO.3, GPIO.4, GPIO.8, J1.2, JMP.2, Q1.E, U1.DVDD, U1.RATE, U1.VSUP; no longer C3.1, C4.1, C7.1, DTR.C, J2.6, R6.1, R7.1, R9.1, RTS.C, RX.C, TX.C, U1.V3, U1.VCC, U2.VCC, U3.OUT, U3.OUT@1
- net GND: now also C1.1, C8.2, C9.1, GPIO.5, GPIO.6, J1.1, LOAD_CELL.2, LOAD_CELL.5, R1.1, R3.2, U1.AGND, U1.INB+, U1.INB-, U1.XI; no longer C1.2, C4.2, J1.GND, J1.SHIELD, J2.1, R8.2, U1.GND, U2.GND, U3.ADJ
- net N$3: now also C5.1, C6.1, L1.1, LOAD_CELL.1; no longer R4.1, RX.A
- net N$4: now also Q1.B, U1.BASE; no longer R5.1, TX.A
Other:
- moved on the sheet: C1, C2, C3, C4, C5, C6, C7, R2, R3, R4, R5, R6
