File: eagle/projects/static_platform_v1.1/StaticPlatformMain_v1.sch (EAGLE design)
At the start: 27 parts, among them J1 1734035-4, U1 HX711, U2 LM393, U3 AMS1117, X1 CSM-7X-DU

Commit message: 150324
Parts:
- removed DTR, RTS, RX, TX: PWR, led:LEDCHIPLED_0805
- removed U$1: DIPSW4, dipsw:DIPSW4
- removed U3: AMS1117, SparkFun-IC-Power:V_REG_LM1117SOT223
- added C10: 10u, rcl:C-EUC0805
- added C11, C12, C13, C14, C15, C16: 100n, rcl:C-EUC0805
- added C8, C9: 1u, 6.3V, rcl:C-EUC0805
- added CR1, CR2: USBLC6-2SC6, usblc6:USBLC6-2SC6
- added FB1, FB2, FB3: 150R 74279207, FB_74279207:74279207
- added GPIO, PROGRAMMING: (no value), SparkFun-Connectors:CONN_05NO_SILK
- added J3, J4: DS1013-10SSIB1, IDC_CON_DS1013-10SSIB1:DS1013-10SSIB1
- added J5: USB_B_PTH, SparkFun-Connectors:USB_B_PTH
- added J6: USB4800-03-A, USB4800-03-A:USB4800-03-A
- added J7: (no value), con-lstb_round_pads:MA03-1
- added JTAG: CORTEX_DEBUG_SMD, SparkFun-Connectors:CORTEX_DEBUG_SMD
- added LED: RED, adafruit:LEDCHIPLED_0805
- added PANEL: S3B-XH-A(LF)(SN), S6B-XH-A_LF__SN_:S3B-XH-A(LF)(SN)
- added PWR: GREEN, adafruit:LEDCHIPLED_0805
- added R10: 1k, rcl:R-EU_R0805
- added R14, R15: 5k1, rcl:R-EU_R0805
- added RESET: MOMENTARY-SWITCH-SPST-SMD-6.0X3.5MM, SparkFun-Switches:MOMENTARY-SWITCH-SPST-SMD-6.0X3.5MM
- added U4: MCP9700TT, SparkFun-Sensors:MCP9700TT
- C1: value 10u -> 1u, 6.3V; device rcl:C-EUC0805K -> rcl:C-EUC0805
- C2: value 5u6 -> 10u, 6.3V; device rcl:C-EUC0805K -> rcl:C-EUC0805
- C3: value 100n -> 4.7u, 6.3V; device rcl:C-EUC0805K -> rcl:C-EUC0805
- C4: value 10n -> 1u, 6.3V; device rcl:C-EUC0805K -> rcl:C-EUC0805
- C5: value 22p -> 100n, 6.3V; device rcl:C-EUC0805K -> rcl:C-EUC0805
- C6: value 22p -> 15p, 6.3V; device rcl:C-EUC0805K -> rcl:C-EUC0805
- C7: value 100n -> 15p, 6.3V; device rcl:C-EUC0805K -> rcl:C-EUC0805
- D1: value BAT60B -> 3A/10V/280mV; device diode:MBR0520LT -> SparkFun-DiscreteSemi:DIODE-SCHOTTKY-BAT60A
- J1: value 1734035-4 -> DS1013-10SSIB1; device USB connector:1734035-4 -> IDC_CON_DS1013-10SSIB1:DS1013-10SSIB1
- J2: value (none) -> DS1013-10SSIB1; device con-lstb_round_pads:MA06-1 -> IDC_CON_DS1013-10SSIB1:DS1013-10SSIB1
- R5, R6, R7, R8: value 1k -> 10k
- U1: value HX711 -> ATSAMD21E18A-AUTQFP32_MC_MCH-M; device ch340:CH340G -> SAMD21E18:ATSAMD21E18A-AUTQFP32_MC_MCH-M
- U2: value LM393 -> AMS1117; device lm393:LM393 -> SparkFun-IC-Power:V_REG_LM1117SOT223
- X1: value CSM-7X-DU -> 32.768kHz; device crystal:CSM-7X-DU -> adafruit:XTAL-3.2X1.5
Connections:
- removed net /DTR: R6.2, U$1.2A, U2.OUTA
- removed net /RTS: R7.2, U$1.4A, U2.OUTB
- removed net CTS: U1.CTS
- removed net DCD: U1.DCD
- removed net DSR: U1.DSR
- removed net DTR: U$1.1A, U1.DTR, U2.INNA
- removed net DTR_O: J2.5, R3.2, U$1.1B, U$1.2B
- removed net D_N: J1.D-, U1.UDN
- removed net D_P: J1.D+, U1.UDP
- removed net N$3: R4.1, RX.A
- removed net N$4: R5.1, TX.A
- removed net RI: U1.RI
- removed net RS232: U1.R232
- removed net RTS: U$1.3A, U1.RTS, U2.INNB
- removed net RTS_O: J2.4, R2.2, U$1.3B, U$1.4B
- removed net RX: J2.3, R4.2, U1.RXD
- removed net TX: J2.2, R5.2, U1.TXD
- removed net USB_5V: C1.1, D1.C, U3.IN
- removed net VBUS: D1.A, J1.VBUS
- removed net VCC/2: R8.1, R9.2, U2.INPA, U2.INPB
- removed net XI: C5.1, U1.XI, X1.2
- removed net XO: C6.1, U1.XO, X1.1
- new net 3V1: R3.2, U1.PA07
- new net 3V3DISP: C16.1, FB3.2, PANEL.6
- new net 5V: C2.1, D1.C, GPIO.1, U2.IN
- new net CC1: J6.CC1, R14.2
- new net CC2: J6.CC2, R15.2
- new net DTCT: JTAG.GNDDTCT
- new net KEY: JTAG.KEY
- new net LC1_CON: J1.9, U1.PA27
- new net LC1_DOUT: J1.5, U1.PA18
- new net LC1_GPIO: J1.3, U1.PA02
- new net LC1_SCK: J1.7, U1.PA19
- new net LC2_CON: J2.9, U1.PA23
- new net LC2_DOUT: J2.5, U1.PA14
- new net LC2_GPIO: J2.3, U1.PA03
- new net LC2_SCK: J2.7, U1.PA15
- new net LC3_CON: J4.9, U1.PA28
- new net LC3_DOUT: J4.5, U1.PA16
- new net LC3_GPIO: J4.3, U1.PA04
- new net LC3_SCK: J4.7, U1.PA17
- new net LC4_CON: J3.9, U1.PA22
- new net LC4_DOUT: J3.5, U1.PA10
- new net LC4_GPIO: J3.3, U1.PA05
- new net LC4_SCK: J3.7, U1.PA11
- new net LED_GP: LED.A, PANEL.2, R3.1
- new net LED_PWR: PANEL.3, PWR.A, R2.1
- new net N$13: J1.4
- new net N$16: J1.6
- new net N$24: JTAG.NC/TDI
- new net N$28: J2.4
- new net N$29: J2.6
- new net N$38: J4.4
- new net N$39: J4.6
- new net N$48: J3.4
- new net N$49: J3.6
- new net N$6: C1.1, U1.VDDCORE
- new net N$8: R4.1, U4.VO
- new net RESET: JTAG.!RESET, PROGRAMMING.2, R7.1, RESET.1, U1.!RESET
- new net SCL: GPIO.5, J1.10, J2.10, J3.10, J4.10, R10.1, R6.1, U1.PA09
- new net SDA: GPIO.4, J1.8, J2.8, J3.8, J4.8, R5.1, R9.1, U1.PA08
- new net SWCLK: JTAG.SWDCLK/TCK, PROGRAMMING.3, R8.1, U1.PA30
- new net SWDIO: JTAG.SWDIO/TMS, PROGRAMMING.4, U1.PA31
- new net SWO: JTAG.SWO/TDO
- new net TS: C9.1, R4.2, U1.PA06
- new net USB_D_N: CR1.I/O1, CR1.I/O1_2, CR2.I/O2, CR2.I/O2_2, J5.D-, J6.DN1, J6.DN2, U1.PA24
- new net USB_D_P: CR1.I/O2, CR1.I/O2_2, CR2.I/O1, CR2.I/O1_2, J5.D+, J6.DP1, J6.DP2, U1.PA25
- new net VBUSC: C11.1, CR2.VBUS, FB1.1, J6.VBUS_1, J6.VBUS_2
- new net VBUSD: C13.1, CR1.VBUS, FB2.1, J5.VBUS
- new net VBUSFC: C12.1, FB1.2, J7.1
- new net VBUSFD: C14.1, FB2.2, J7.3
- new net VBUSOUT: D1.A, J7.2
- new net XTAL1: C6.2, U1.PA00, X1.P$1
- new net XTAL2: C7.2, U1.PA01, X1.P$2
- net 3V3: now also C10.1, C15.1, C5.1, C8.2, FB3.1, GPIO.2, J1.2, J2.2, J3.2, J4.2, JTAG.VCC, PROGRAMMING.5, R2.2, R5.2, R6.2, R7.2, R8.2, U1.VDDANA, U1.VDDIN, U2.OUT, U2.OUT@1, U4.VCC; no longer C2.1, C7.1, DTR.C, J2.6, R6.1, R7.1, R9.1, RTS.C, RX.C, TX.C, U1.V3, U1.VCC, U2.VCC, U3.OUT, U3.OUT@1
- net GND: now also C10.2, C11.2, C12.2, C13.2, C14.2, C15.2, C16.2, C6.1, C7.1, C8.1, C9.2, CR1.GND, CR2.GND, GPIO.3, J1.1, J3.1, J4.1, J5.GND, J5.SHIELD, J6.GND_1, J6.GND_2, J6.MH3, J6.MH4, J6.MH5, J6.MH6, JTAG.GND@3, JTAG.GND@5, LED.C, PANEL.1, PROGRAMMING.1, PWR.C, R14.1, R15.1, RESET.2, U1.GND_2, U2.ADJ, U4.GND; no longer C6.2, C7.2, J1.GND, J1.SHIELD, R8.2, U2.GND, U3.ADJ
- net N$1: now also PANEL.5, R10.2; no longer DTR.A, R3.1
- net N$2: now also PANEL.4, R9.2; no longer R2.1, RTS.A
Other:
- note added: "1.1"
- note added: "CONNECTORS"
- note added: "Designed by Yusuf Atalay"
- note added: "INPUT STAGE"
- note added: "Rev: A.U."
- note added: "Revision Notes 1.1: 03.2023, Abdurrahman ÜZÜM 1- Rerouted the board, removed smoothed tracks and unnecessary jumps, brought groups of pins closer, ensured uninterrupted ground pours beneath USB pairs and oscillator. 2- Updated DRC to meet the local manufacturing requirements. 3- Added standard 10 pin 0.127mm pitch JTAG header. 4- Added USB Type-C (USB2.0, 16 pin) port. 5- Added thermal isolation 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"
- note added: "Static Platform Main"
- note added: "TEMPERATURE SENSOR"
- note added: "uCONTROLLER"
- moved on the sheet: C1, C2, C3, C4, C5, C6, C7, R2, R3, R4, R5, R6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
