File: eagle/projects/double_pulse_timer/timer.brd (EAGLE design)
At the start: 29.2 x 54.7 mm, 13 parts, among them IC1 74HC02N, Q1 VN10KM

Commit message: 260524
Routing:
- net N$3: track 6.66 -> 8.15 mm
- net N$4: track 6.66 -> 8.15 mm
Changed lines of the file:
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@@
 <contactref element="R11" pad="1"/>
 <contactref element="D1" pad="A"/>
-<wire x1="67.31" y1="50.8" x2="71.12" y2="54.61" width="0.8128" layer="1"/>
-<wire x1="71.12" y1="54.61" x2="71.12" y2="55.88" width="0.8128" layer="1"/>
+<wire x1="71.12" y1="52.07" x2="69.85" y2="50.8" width="0.8128" layer="1"/>
+<wire x1="67.31" y1="50.8" x2="69.85" y2="50.8" width="0.8128" layer="1"/>
+<wire x1="71.12" y1="52.07" x2="71.12" y2="55.88" width="0.8128" layer="1"/>
 </signal>
 <signal name="N$4">
 <contactref element="D2" pad="C"/>
 <contactref element="R12" pad="1"/>
-<wire x1="74.93" y1="50.8" x2="78.74" y2="54.61" width="0.8128" layer="1"/>
-<wire x1="78.74" y1="54.61" x2="78.74" y2="55.88" width="0.8128" layer="1"/>
+<wire x1="78.74" y1="52.07" x2="77.47" y2="50.8" width="0.8128" layer="1"/>
+<wire x1="74.93" y1="50.8" x2="77.47" y2="50.8" width="0.8128" layer="1"/>
+<wire x1="78.74" y1="52.07" x2="78.74" y2="55.88" width="0.8128" layer="1"/>
 </signal>
 <signal name="N$5">
